File: KiCad/Compucorp_324G_Keyboard.kicad_sch (KiCad schematic)
At the start: 49 parts, among them J3 To Scan Board, SW1 e^x 10^x, SW10 2nd FUNC, SW11 ARCTAN, SW12 a^x, SW13 5, SW14 EXCHn, SW15 START/STOP, SW16 x,y → Θ,r, SW17 DIV, SW18 EXP, SW19 4, SW2 ), SW20 RCLn, SW21 CLEAR ENTRY, SW22 º → R → º, SW23 ARCSIN ARCCOS, SW24 MUL, SW25 CHG SIGN, SW26 3, SW27 STn, SW28 RESET, SW29 TAN, SW3 DEC → D.MS, SW30 INV, SW31 MINUS, SW32 DP, SW33 2, SW34 Θ,r → x,y, SW35 SQRT, SW36 PLUS, SW37 9, SW38 1, SW39 SIN COS, SW4 7, SW40 PI, SW41 EQUALS, SW42 8, SW43 0, SW44 UNKNOWN, SW45 RUN/LOAD, SW46 PROG 1/2, SW47 RUN/STEP/LOAD, SW48 GRAD/DEG, SW5 Ln LOG, SW6 (, SW7 D.MS → DEC, SW8 6, SW9 SET DP

Commit message: Updated keyboard schematic
Parts:
- SW44: value UNKNOWN -> FED/MUNI
Connections:
- net Col 1 renamed KB Col 1
- net Col 2 renamed KB Col 2
- net Col 3 renamed KB Col 3
- net Col 4 renamed KB Col 4
- net Col 5 renamed KB Col 5
- net Col 6 renamed KB Col 6
- net Col 7 renamed KB Col 7
- net Col 8 renamed KB Col 8
- net Col 9 renamed KB Col 9
- net GRAD renamed KB GRAD
- net LOAD renamed KB LOAD
- net PROG 1 renamed KB PROG 1
- net Pin 20 renamed TCL02 Pin 38
- net Pin 21 renamed KB FED
- net RUN renamed KB RUN
- net Row 1 renamed KB Row 1
- net Row 2 renamed KB Row 2
- net Row 3 renamed KB Row 3
- net Row 4 renamed KB Row 4
- net Row 5 renamed KB Row 5
- net Row 6 renamed KB Row 6
- net Row 7 renamed KB Row 7
- net Row 8 renamed KB Row 8
Other:
- moved on the sheet: SW44, SW45, SW46, SW47, SW48
