File: KiCad/Compucorp_324G_Memory_Board.kicad_sch (KiCad schematic)
At the start: 37 parts, among them J10 Memory Interboard, Q1 2N4403, Q2 2N4403, Q3 2N4403, Q4 2N4403, U10 2102, U11 2102, U12 2102, U13 93L00, U14 93L00, U15 93L00, U16 74L75, U17 TMC1871 (TCL03), U18 8KR11A, U19 8KR029, U20 8KR218, U9 2102

Commit message: Update Compucorp_324G_Memory_Board.kicad_sch
Connections:
- net IB_24: now reaches J10.a24 (Pin_a24)
- net IB_24: now also J10.b24 (Pin_b24)
- net IB_21: now reaches J10.b21 (Pin_b21)
- no-connect marks 71 -> 69
Changed lines of the file:
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@@
 	)
 	(no_connect
-		(at 373.38 194.31)
-	)
-	(no_connect
-		(at 386.08 194.31)
-	)
-	(no_connect
 		(at 201.93 109.22)
 	)
@@
 		)
 	)
+	(global_label "IB_21"
+		(shape input)
+		(at 386.08 186.69 0)
+		(fields_autoplaced yes)
+		(effects
+			(font
+				(size 1.27 1.27)
+			)
+			(justify left)
+		)
+		(property "Intersheetrefs" "${INTERSHEET_REFS}"
+			(at 394.3266 186.69 0)
+			(effects
+				(font
+					(size 1.27 1.27)
+				)
+				(justify left)
+				(hide yes)
+			)
+		)
+	)
 	(global_label "IB_14"
 		(shape input)
@@
 		)
 	)
+	(global_label "IB_24"
+		(shape input)
+		(at 373.38 194.31 180)
+		(fields_autoplaced yes)
+		(effects
+			(font
+				(size 1.27 1.27)
+			)
+			(justify right)
+		)
+		(property "Intersheetrefs" "${INTERSHEET_REFS}"
+			(at 365.1334 194.31 0)
+			(effects
+				(font
+					(size 1.27 1.27)
+				)
+				(justify right)
+				(hide yes)
+			)
+		)
+	)
 	(global_label "IB_07"
 		(shape input)
@@
 				(hide yes)
 			)
+		)
+	)
+	(global_label "IB_24"
+		(shape input)
+		(at 386.08 194.31 0)
+		(fields_autoplaced yes)
+		(effects
+			(font
+				(size 1.27 1.27)
+			)
+			(justify left)
+		)
+		(property "Intersheetrefs" "${INTERSHEET_REFS}"
+			(at 394.3266 194.31 0)
+			(effects
+				(font
+					(size 1.27 1.27)
+				)
+				(justify left)
+				(hide yes)
+			)

Commit message: Update Compucorp_324G_Memory_Board.kicad_sch
Connections:
- net IB_39: no longer J10.b39 (Pin_b39)
- no-connect marks 69 -> 70
Changed lines of the file:
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@@
 		)
 	)
+	(text_box "Guesses ...\n\nIB07 = Data from ROM/RAM\nIB08 = Data from ROM/RAM\nIB09 = Data from ROM/RAM\nIB10 = Data from ROM/RAM\n\nIB28 = Data to RAM\nIB29 = Data to RAM\nIB30 = Data to RAM\nIB31 = Data to RAM\n\nTCL03_08 = A_{0}\nTCL03_30 = A_{1}\nTCL03_29 = A_{2}\nTCL03_28 = A_{3}\nTCL03_21 = A_{4}\nTCL03_26 = A_{5}\nTCL03_25 = A_{6}\nTCL03_24 = A_{7}\nTCL03_23 = A_{8}\nTCL03_18 = A_{9}\nTCL03_11 = RAM CE\n"
+		(exclude_from_sim no)
+		(at 259.08 182.88 0)
+		(size 36.83 49.53)
+		(margins 0.9525 0.9525 0.9525 0.9525)
+		(stroke
+			(width 0)
+			(type solid)
+		)
+		(fill
+			(type none)
+		)
+		(effects
+			(font
+				(size 1.27 1.27)
+			)
+			(justify left top)
+		)
+	)
 	(junction
 		(at 129.54 228.6)
@@
 	)
 	(no_connect
+		(at 386.08 232.41)
+	)
+	(no_connect
 		(at 386.08 209.55)
 	)
@@
 				(hide yes)
 			)
-		)
-	)
-	(global_label "IB_39"
-		(shape input)
-		(at 386.08 232.41 0)
-		(fields_autoplaced yes)
-		(effects
-			(font
-				(size 1.27 1.27)
-			)
-			(justify left)
-		)
-		(property "Intersheetrefs" "${INTERSHEET_REFS}"
-			(at 394.3266 232.41 0)
-			(effects
-				(font
-					(size 1.27 1.27)
-				)
-				(justify left)
-				(hide yes)
-			)

Commit message: Update Compucorp_324G_Memory_Board.kicad_sch
Parts:
- removed U18: 8KR11A, symbol Compucorp_324G_Scientist:ROM
- removed U19: 8KR029, symbol Compucorp_324G_Scientist:ROM
- removed U20: 8KR218, symbol Compucorp_324G_Scientist:ROM
- added U22: 8KR11A, symbol Compucorp_324G_Scientist:8kbit ROM
- added U23: 8KR029, symbol Compucorp_324G_Scientist:8kbit ROM
- added U24: 8KR218, symbol Compucorp_324G_Scientist:8kbit ROM
- renumbered R15 to R19, R6 to R20, R4 to R21, R5 to R22, U16 to Z10, U12 to Z11, U11 to Z12, U10 to Z13, U9 to Z14, U13 to Z7, U14 to Z8, U15 to Z9
Connections:
- net IB_33 is gone; now on net Φ2: J10.a33 (Pin_a33), J10.b33 (Pin_b33), U17.37 (Pin_37), Z10.13 (E01), Z10.4 (E23)
- net TCL03_05 is gone; now on net V_{GG}: U17.5 (Pin_5)
- net TCL03_27 is gone; now on net A4: U17.27 (Pin_27)
- net IB_15: no longer J10.b15 (Pin_b15), U17.2 (Pin_2)
- net Φ2: now reaches Z8.10 (CP)
- net Φ2: now also Z7.10 (CP), Z9.10 (CP)
- net at Q2.2 (B), R16.2: now also R17.2
- net +5V renamed V_{SS}
- net V_{SS}: now also U22.1 (V_{SS}), U23.1 (V_{SS}), U24.1 (V_{SS})
- net -10V renamed V_{DD}
- net V_{DD}: now also U22.28 (V_{DD}), U23.28 (V_{DD}), U24.28 (V_{DD})
- net -25V renamed V_{GG}
- net V_{GG}: now also U22.19 (V_{GG}), U23.19 (V_{GG}), U24.19 (V_{GG})
- net IB_01 renamed CTRL
- net IB_05 renamed C08P
- net IB_06 renamed C16P
- net IB_07 renamed MO2
- net MO2: now also U22.22 (DO2), U23.22 (DO2), U24.22 (DO2)
- net IB_08 renamed MO1
- net MO1: now also U22.23 (DO1), U23.23 (DO1), U24.23 (DO1)
- net IB_09 renamed MO8
- net MO8: now also U22.20 (DO8), U23.20 (DO8), U24.20 (DO8)
- net IB_10 renamed MO4
- net MO4: now also U22.21 (DO4), U23.21 (DO4), U24.21 (DO4)
- net IB_17 renamed ΦR
- net ΦR: now also U22.3 (ΦR), U23.3 (ΦR), U24.3 (ΦR)
- net IB_24 renamed ~{INL2}
- net IB_28 renamed MI1
- net IB_29 renamed MI2
- net IB_30 renamed MI4
- net IB_31 renamed MI8
- net IB_32 renamed Φ1
- net Φ1: now also U22.2 (Φ1), U23.2 (Φ1), U24.2 (Φ1)
- net RAM_A_{0} renamed A0D
- net RAM_A_{1} renamed A1D
- net RAM_A_{2} renamed A2D
- net RAM_A_{3} renamed A3D
- net RAM_A_{4} renamed A4D
- net RAM_A_{5} renamed A5D
- net RAM_A_{6} renamed A6D
- net RAM_A_{7} renamed A7D
- net RAM_A_{8} renamed A8D
- net RAM_A_{9} renamed A_{9}D
- net A_{9}D: no longer Z9.14 (Q1)
- net RAM_CE renamed ~{CTEND}
- net RAM_D_{IN1} renamed ~{DI8}
- net RAM_D_{IN2} renamed ~{DI4}
- net RAM_D_{IN3} renamed ~{DI2}
- net RAM_D_{IN4} renamed ~{DI1}
- net RAM_D_{OUT1} renamed ~{DO8}
- net RAM_D_{OUT2} renamed ~{DO4}
- net RAM_D_{OUT3} renamed ~{DO2}
- net RAM_D_{OUT4} renamed ~{DO1}
- net RAM_RW renamed R/W
- net TCL03_08 renamed A0
- net A0: now also U22.4 (A0), U23.4 (A0), U24.4 (A0)
- net TCL03_09 renamed A14
- net A14: now also U22.27 (A14), U23.27 (A14), U24.27 (A14)
- net TCL03_10 renamed A13
- net A13: now also U22.26 (A13), U23.26 (A13), U24.26 (A13)
- net TCL03_11 renamed ~{CTEN}
- net TCL03_13 renamed A12
- net A12: now also U22.25 (A12), U23.25 (A12), U24.25 (A12)
- net TCL03_14 renamed A11
- net A11: now also U22.24 (A11), U23.24 (A11), U24.24 (A11)
- net TCL03_17 renamed A10
- net A10: now also U22.18 (A10), U23.18 (A10), U24.18 (A10)
- net TCL03_18 renamed A9
- net A9: now also U22.17 (A9), U23.17 (A9), U24.17 (A9)
- net TCL03_21 renamed A4
- net A4: now also U22.8 (A4), U23.8 (A4), U24.8 (A4)
- net TCL03_23 renamed A8
- net A8: now also U22.12 (A8), U23.12 (A8), U24.12 (A8)
- net TCL03_24 renamed A7
- net A7: now also U22.11 (A7), U23.11 (A7), U24.11 (A7)
- net TCL03_25 renamed A6
- net A6: now also U22.10 (A6), U23.10 (A6), U24.10 (A6)
- net TCL03_26 renamed A5
- net A5: now also U22.9 (A5), U23.9 (A5), U24.9 (A5)
- net TCL03_28 renamed A3
- net A3: now also U22.7 (A3), U23.7 (A3), U24.7 (A3)
- net TCL03_29 renamed A2
- net A2: now also U22.6 (A2), U23.6 (A2), U24.6 (A2)
- net TCL03_30 renamed A1
- net A1: now also U22.5 (A1), U23.5 (A1), U24.5 (A1)
- new net A9D: Z9.14 (Q1)
- new net WRIT: J10.b15 (Pin_b15), U17.2 (Pin_2)
- no-connect marks 70 -> 67
Other:
- moved on the sheet: R17
