File: KiCad/Compucorp_324G_Scan_Board.kicad_sch (KiCad schematic)
At the start: 24 parts, among them J1 Scan Interboard, J2 Power In, J4 From Keyboard, U1 BR 16252, U2 UHP480, U21 TMC1884 (TCL08), U3 UHP480, U4 TMC1869 (TCL02)

Commit message: Update Compucorp_324G_Scan_Board.kicad_sch
Parts:
- added D13, D14, D15, D16, D17, D18: D, symbol Device:D
- added JP1: E1-E2, symbol Jumper:SolderJumper_2_Bridged
Connections:
- net IB_01: now also U21.34 (Pin_34), U4.5 (Pin_5)
- net KB Col 1: now also U4.26 (Pin_26)
- net KB Col 5: now also U4.27 (Pin_27)
- net KB Col 6: now also U4.30 (Pin_30)
- net KB GRAD: now also JP1.2 (B)
- net KB PROG 1: now also D15.2 (A)
- net KB RUN: now also D6.2 (A), D13.2 (A)
- net KB Row 1: now also U4.20 (Pin_20)
- net KB Row 2: now also U4.18 (Pin_18)
- net KB Row 3: now also D14.2 (A)
- net KB Row 4: now also D16.2 (A)
- net KB Row 7: now also D7.2 (A)
- net TCL02_10: now reaches D3.1 (K)
- net TCL02_10: now also D4.1 (K), U4.10 (Pin_10)
- net TCL02_06: now reaches D8.1 (K)
- net TCL02_06: now also D5.1 (K), U4.6 (Pin_6), D18.1 (K)
- net TCL02_12: now reaches D2.1 (K)
- net TCL02_12: now also D1.1 (K), U4.12 (Pin_12), D17.1 (K)
- net TCL02_08: now reaches D7.1 (K)
- net TCL02_08: now also D6.1 (K), U4.8 (Pin_8), JP1.1 (A)
- net TCL02_14: now reaches U4.14 (Pin_14)
- net TCL02_14: now also D14.1 (K), D16.1 (K)
- net TCL02_16: now reaches U4.16 (Pin_16)
- net TCL02_16: now also D13.1 (K), D15.1 (K)
- net TCL02_37: now reaches U4.37 (Pin_37)
- net TCL02_37: now also D17.2 (A), D18.2 (A)
Other:
- moved on the sheet: J4

Commit message: Update Compucorp_324G_Scan_Board.kicad_sch
Connections:
- net KB Col 1 renamed KB_COL_1
- net KB Col 2 renamed KB_COL_2
- net KB Col 3 renamed KB_COL_3
- net KB Col 4 renamed KB_COL_4
- net KB Col 5 renamed KB_COL_5
- net KB Col 6 renamed KB_COL_6
- net KB Col 7 renamed KB_COL_7
- net KB Col 8 renamed KB_COL_8
- net KB Col 9 renamed KB_COL_9
- net KB FED renamed KB_FED
- net KB GRAD renamed KB_GRAD
- net KB LOAD renamed KB_LOAD
- net KB PROG 1 renamed KB_PROG 1
- net KB_PROG 1: no longer J4.6 (Pin_6)
- net KB RUN renamed KB_RUN
- net KB_RUN: no longer D13.2 (A), J4.23 (Pin_23)
- net KB Row 1 renamed KB_ROW_1
- net KB Row 2 renamed KB_ROW_2
- net KB Row 3 renamed KB_ROW_3
- net KB Row 4 renamed KB_ROW_4
- net KB Row 5 renamed KB_ROW_5
- net KB Row 6 renamed KB_ROW_6
- net KB Row 7 renamed KB_ROW_7
- net KB Row 8 renamed KB_ROW_8
- new net KB_PROG_1: J4.6 (Pin_6)
- new net KB_RUN_{326}: D13.2 (A), J4.23 (Pin_23)
Changed lines of the file:
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@@
 		)
 	)
-	(global_label "KB Col 8"
+	(global_label "KB_COL_8"
 		(shape input)
 		(at 120.65 105.41 180)
@@
 		)
 	)
-	(global_label "KB Row 3"
+	(global_label "KB_ROW_3"
 		(shape input)
 		(at 120.65 69.85 180)
@@
 		)
 	)
-	(global_label "KB Col 6"
+	(global_label "KB_COL_6"
 		(shape input)
 		(at 68.58 87.63 0)
@@
 		)
 	)
-	(global_label "KB Row 6"
+	(global_label "KB_ROW_6"
 		(shape input)
 		(at 120.65 128.27 180)
@@
 		)
 	)
-	(global_label "KB GRAD"
+	(global_label "KB_GRAD"
 		(shape input)
 		(at 120.65 123.19 180)
@@
 		)
 	)
-	(global_label "KB Row 1"
+	(global_label "KB_ROW_1"
 		(shape input)
 		(at 120.65 64.77 180)
@@
 		)
 	)
-	(global_label "KB Col 3"
+	(global_label "KB_COL_3"
 		(shape input)
 		(at 120.65 82.55 180)
@@
 		)
 	)
-	(global_label "KB Col 1"
+	(global_label "KB_COL_1"
 		(shape input)
 		(at 120.65 80.01 180)
@@
 		)
 	)
-	(global_label "KB LOAD"
+	(global_label "KB_LOAD"
 		(shape input)
 		(at 120.65 190.5 180)
@@
 		)
 	)
-	(global_label "KB GRAD"
+	(global_label "KB_GRAD"
 		(shape input)
 		(at 120.65 152.4 180)
@@
 		)
 	)
-	(global_label "KB Col 1"
+	(global_label "KB_COL_1"
 		(shape input)
 		(at 68.58 97.79 0)
@@
 		)
 	)
-	(global_label "KB GRAD"
+	(global_label "KB_GRAD"
 		(shape input)
 		(at 143.51 200.66 0)
@@
 		)
 	)
-	(global_label "KB Row 8"
+	(global_label "KB_ROW_8"
 		(shape input)
 		(at 120.65 133.35 180)
@@
 		)
 	)
-	(global_label "KB Row 1"
+	(global_label "KB_ROW_1"
 		(shape input)
 		(at 43.18 110.49 180)
@@
 		)
 	)
-	(global_label "KB Col 7"
+	(global_label "KB_COL_7"
 		(shape input)
 		(at 68.58 80.01 0)
@@
 		)
 	)
-	(global_label "KB Row 3"
+	(global_label "KB_ROW_3"
 		(shape input)
 		(at 120.65 173.99 180)
@@
 		)
 	)
-	(global_label "KB Col 5"
+	(global_label "KB_COL_5"
 		(shape input)
 		(at 120.65 85.09 180)
@@
 		)
 	)
-	(global_label "KB Col 4"
+	(global_label "KB_COL_4"
 		(shape input)
 		(at 120.65 90.17 180)
@@
 		)
 	)
-	(global_label "KB Col 9"
+	(global_label "KB_COL_9"
 		(shape input)
 		(at 68.58 74.93 0)
@@
 		)
 	)
-	(global_label "KB PROG 1"
+	(global_label "KB_PROG_1"
 		(shape input)
 		(at 120.65 77.47 180)
@@
 		)
 	)
-	(global_label "KB RUN"
+	(global_label "KB_RUN_{326}"
 		(shape input)
 		(at 120.65 181.61 180)
@@
 		)
 		(property "Intersheetrefs" "${INTERSHEET_REFS}"
-			(at 110.2262 181.61 0)
-			(effects
-				(font
-					(size 1.27 1.27)
-				)
-				(justify right)
-				(hide yes)
-			)
-		)
-	)
-	(global_label "KB Col 9"
+			(at 107.2726 181.61 0)
+			(effects
+				(font
+					(size 1.27 1.27)
+				)
+				(justify right)
+				(hide yes)
+			)
+		)
+	)
+	(global_label "KB_COL_9"
 		(shape input)
 		(at 120.65 107.95 180)
@@
 		)
 	)
-	(global_label "KB FED"
+	(global_label "KB_FED"
 		(shape input)
 		(at 120.65 115.57 180)
@@
 		)
 	)
-	(global_label "KB FED"
+	(global_label "KB_FED"
 		(shape input)
 		(at 120.65 157.48 180)
@@
 		)
 	)
-	(global_label "KB Col 5"
+	(global_label "KB_COL_5"
 		(shape input)
 		(at 68.58 95.25 0)
@@
 		)
 	)
-	(global_label "KB LOAD"
+	(global_label "KB_LOAD"
 		(shape input)
 		(at 120.65 118.11 180)
@@
 		)
 	)
-	(global_label "KB RUN"
+	(global_label "KB_RUN"
 		(shape input)
 		(at 116.84 200.66 180)
@@
 		)
 	)
-	(global_label "KB RUN"
+	(global_label "KB_RUN"
 		(shape input)
 		(at 120.65 74.93 180)
@@
 		)
 	)
-	(global_label "KB Col 8"
+	(global_label "KB_COL_8"
 		(shape input)
 		(at 68.58 77.47 0)
@@
 		)
 	)
-	(global_label "KB Row 5"
+	(global_label "KB_ROW_5"
 		(shape input)
 		(at 120.65 125.73 180)
@@
 		)
 	)
-	(global_label "KB Row 2"
+	(global_label "KB_ROW_2"
 		(shape input)
 		(at 120.65 67.31 180)
@@
 		)
 	)
-	(global_label "KB Row 2"
+	(global_label "KB_ROW_2"
 		(shape input)
 		(at 43.18 105.41 180)
@@
 		)
 	)
-	(global_label "KB Col 2"
+	(global_label "KB_COL_2"
 		(shape input)
 		(at 120.65 92.71 180)
@@
 		)
 	)
-	(global_label "KB Row 4"
+	(global_label "KB_ROW_4"
 		(shape input)
 		(at 120.65 177.8 180)
@@
 		)
 	)
-	(global_label "KB Row 5"
+	(global_label "KB_ROW_5"
 		(shape input)
 		(at 120.65 161.29 180)
@@
 		)
 	)
-	(global_label "KB PROG 1"
+	(global_label "KB_PROG 1"
 		(shape input)
 		(at 120.65 185.42 180)
@@
 		)
 	)
-	(global_label "KB RUN"
+	(global_label "KB_RUN_{326}"
 		(shape input)
 		(at 120.65 120.65 180)
@@
 		)
 		(property "Intersheetrefs" "${INTERSHEET_REFS}"
-			(at 110.2262 120.65 0)
+			(at 107.2726 120.65 0)
 			(effects
 				(font
@@
 		)
 	)
-	(global_label "KB Row 8"
+	(global_label "KB_ROW_8"
 		(shape input)
 		(at 120.65 148.59 180)
@@
 		)
 	)
-	(global_label "KB Col 7"
+	(global_label "KB_COL_7"
 		(shape input)
 		(at 120.65 102.87 180)
@@
 		)
 	)
-	(global_label "KB Row 7"
+	(global_label "KB_ROW_7"
 		(shape input)
 		(at 116.84 204.47 180)
@@
 		)
 	)
-	(global_label "KB Row 6"
+	(global_label "KB_ROW_6"
 		(shape input)
 		(at 120.65 194.31 180)
@@
 		)
 	)
-	(global_label "KB Col 6"
+	(global_label "KB_COL_6"
 		(shape input)
 		(at 120.65 95.25 180)
@@
 		)
 	)
-	(global_label "KB Row 7"
+	(global_label "KB_ROW_7"
 		(shape input)
 		(at 120.65 130.81 180)
@@
 		)
 	)
-	(global_label "KB Row 4"
+	(global_label "KB_ROW_4"
 		(shape input)
 		(at 120.65 72.39 180)

Commit message: Update Compucorp_324G_Scan_Board.kicad_sch
Parts:
- removed D17, D18: D, symbol Device:D
Connections:
- net +5V is gone; now on net V_{SS}: J2.1 (Pin_1)
- net -10V is gone; now on net V_{DD}: J1.b35 (Pin_b35)
- net -25V is gone; now on net V_{GG}: J1.b36 (Pin_b36)
- net IB_24 is gone; now on net ~{INL2}: J1.b24 (Pin_b24)
- net IB_32 is gone; now on net Φ1: J1.b32 (Pin_b32)
- net IB_33 is gone; now on net Φ2: J1.b33 (Pin_b33)
- net KB_COL_2 is gone; now on net Y9: J4.12 (Pin_12)
- net KB_COL_4 is gone; now on net Y6: J4.11 (Pin_11)
- net KB_ROW_7 is gone; now on net KX2: D7.2 (A), J4.27 (Pin_27)
- net KB_RUN is gone; now on net AXB: D6.2 (A), J4.5 (Pin_5)
- net V_{SS}: now reaches U21.1 (V_{SS})
- net V_{SS}: now also U21.2 (~{ADR2}), U21.3 (~{ADR1}), U21.40 (~{TEST}), U4.1 (V_{SS})
- net V_{DD}: now reaches U21.20 (V_{DD})
- net V_{DD}: now also U4.21 (V_{DD})
- net V_{GG}: now reaches U21.21 (V_{GG})
- net V_{GG}: now also U4.22 (V_{GG})
- net Φ1: now reaches U21.22 (Φ1)
- net Φ1: now also U4.23 (Φ1)
- net Φ2: now reaches U21.23 (Φ2)
- net Φ2: now also U4.24 (Φ2)
- net ~{INL8}: now reaches U4.11 (INL8)
- net ~{INH1}: now reaches U4.13 (INH1)
- net ~{INH2}: now reaches U4.15 (INH2)
- net ~{INH4}: now reaches U4.17 (INH4)
- net ~{INH8}: now reaches U4.19 (INH8)
- net IXDI: now reaches U4.4 (TXD1)
- net ~{INL2}: now reaches U4.7 (INL2)
- net ~{INL4}: now reaches U4.9 (INL4)
- net Digit_{10} renamed AN7
- net Digit_{11} renamed AN6
- net Digit_{12} renamed AN5
- net Digit_{13} renamed AN4
- net Digit_{14} renamed AN3
- net Digit_{15} renamed AN2
- net Digit_{16} renamed AN1
- net Digit_{1} renamed AN16
- net Digit_{2} renamed AN15
- net Digit_{3} renamed AN14
- net Digit_{4} renamed AN13
- net Digit_{5} renamed AN12
- net Digit_{6} renamed AN11
- net Digit_{7} renamed AN10
- net Digit_{8} renamed AN9
- net Digit_{9} renamed AN8
- net IB_01 renamed CTRL
- net IB_05 renamed C08P
- net IB_06 renamed C16P
- net IB_07 renamed MO2
- net IB_08 renamed MO1
- net IB_09 renamed MO8
- net IB_10 renamed MO4
- net IB_20 renamed PW0N
- net KB_COL_1 renamed Y9
- net KB_COL_3 renamed Y6
- net KB_COL_5 renamed Y8
- net KB_COL_6 renamed Y5
- net KB_COL_7 renamed Y2
- net KB_COL_8 renamed Y1
- net KB_COL_9 renamed Y0
- net KB_FED renamed AX8
- net AX8: now also D16.2 (A); no longer D1.2 (A)
- net KB_GRAD renamed AX1
- net KB_LOAD renamed AX4
- net KB_PROG 1 renamed AXB
- net KB_PROG_1 renamed AXA
- net AXA: now also D2.2 (A)
- net KB_ROW_1 renamed KXD
- net KB_ROW_2 renamed KXC
- net KB_ROW_3 renamed KX2
- net KX2: no longer J4.3 (Pin_3)
- net KB_ROW_4 renamed KXA
- net KXA: now also D1.2 (A); no longer D16.2 (A)
- net KB_ROW_5 renamed KXB
- net KXB: now also D13.2 (A), J4.3 (Pin_3); no longer D2.2 (A)
- net KB_ROW_6 renamed KX4
- net KB_ROW_8 renamed KX1
- net KB_RUN_{326} renamed AX2
- net AX2: no longer D13.2 (A)
- net K_{a} renamed S_{a}
- net K_{b} renamed S_{b}
- net K_{c} renamed S_{c}
- net K_{d} renamed S_{d}
- net K_{e} renamed S_{e}
- net K_{f} renamed S_{f}
- net K_{g} renamed S_{g}
- net K_{h} renamed DP
- net K_{i} renamed COMMA
- net TCL02_06: no longer names the net of D5.1 (K), D8.1 (K), U4.6 (X1)
- net TCL02_12: no longer names the net of D1.1 (K), D2.1 (K)
- net TCL02_12: now also U4.14 (XA); no longer U4.12 (Pin_12)
- net TCL02_14: no longer names the net of D14.1 (K), D16.1 (K)
- net TCL02_14: now also U4.12 (X8); no longer U4.14 (Pin_14)
- net TCL02_16: no longer names the net of D13.1 (K), D15.1 (K), U4.16 (XB)
- net TCL02_37: no longer names the net of U4.37 (YB)
- net TCL02_38 renamed YA
- no-connect marks 44 -> 49
Other:
- moved on the sheet: U4
